File: Hardware/USB_Breakout_Test_Jig/USB_Breakout_Test_Jig.kicad_sch (KiCad schematic)
At the start: 3 parts, among them U1 ESP32_NODEMCU, U2 DM-OLED096-636

Commit message: WIP
Connections:
- net A - 5V renamed A - 5V (red)
- net A - D+ renamed A - D+ (green)
- net A - D- renamed A - D- (white)
- net A - GND renamed A - GND (black)
- net A - ID renamed A - ID (yellow)
- net A - Shield renamed A - Shield (blue)
- net B - 5V renamed B - 5V (red)
- net B - D+ renamed B - D+ (green)
- net B - D- renamed B - D-b(white)
- net B - GND renamed B - GND (black)
- net B - ID renamed B - ID (yellow)
- net B - Shield renamed B - Shield (blue)
Changed lines of the file:
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@@
     (stroke (width 0) (type default))
   )
-  (global_label "B - GND" (shape input) (at 147.32 83.82 0) (fields_autoplaced)
+  (global_label "B - GND (black)" (shape input) (at 147.32 83.82 0) (fields_autoplaced)
     (effects (font (size 1.27 1.27)) (justify left))
-    (property "Intersheetrefs" "${INTERSHEET_REFS}" (at 158.9533 83.82 0)
+    (property "Intersheetrefs" "${INTERSHEET_REFS}" (at 166.6942 83.82 0)
       (effects (font (size 1.27 1.27)) (justify left) hide)
     )
   )
-  (global_label "A - D-" (shape input) (at 147.32 59.69 0) (fields_autoplaced)
+  (global_label "A - D- (white)" (shape input) (at 147.32 59.69 0) (fields_autoplaced)
     (effects (font (size 1.27 1.27)) (justify left))
-    (property "Intersheetrefs" "${INTERSHEET_REFS}" (at 157.7438 59.69 0)
+    (property "Intersheetrefs" "${INTERSHEET_REFS}" (at 165.3034 59.69 0)
       (effects (font (size 1.27 1.27)) (justify left) hide)
     )
   )
-  (global_label "B - D+" (shape input) (at 147.32 95.25 0) (fields_autoplaced)
+  (global_label "B - D+ (green)" (shape input) (at 147.32 95.25 0) (fields_autoplaced)
     (effects (font (size 1.27 1.27)) (justify left))
-    (property "Intersheetrefs" "${INTERSHEET_REFS}" (at 157.9252 95.25 0)
+    (property "Intersheetrefs" "${INTERSHEET_REFS}" (at 165.8476 95.25 0)
       (effects (font (size 1.27 1.27)) (justify left) hide)
     )
   )
-  (global_label "B - 5V" (shape input) (at 147.32 87.63 0) (fields_autoplaced)
+  (global_label "B - 5V (red)" (shape input) (at 147.32 87.63 0) (fields_autoplaced)
     (effects (font (size 1.27 1.27)) (justify left))
-    (property "Intersheetrefs" "${INTERSHEET_REFS}" (at 157.3809 87.63 0)
+    (property "Intersheetrefs" "${INTERSHEET_REFS}" (at 163.0657 87.63 0)
       (effects (font (size 1.27 1.27)) (justify left) hide)
     )
   )
-  (global_label "A - ID" (shape input) (at 147.32 67.31 0) (fields_autoplaced)
+  (global_label "A - ID (yellow)" (shape input) (at 147.32 67.31 0) (fields_autoplaced)
     (effects (font (size 1.27 1.27)) (justify left))
-    (property "Intersheetrefs" "${INTERSHEET_REFS}" (at 156.7762 67.31 0)
+    (property "Intersheetrefs" "${INTERSHEET_REFS}" (at 165.3033 67.31 0)
       (effects (font (size 1.27 1.27)) (justify left) hide)
     )
   )
-  (global_label "A - GND" (shape input) (at 147.32 52.07 0) (fields_autoplaced)
+  (global_label "A - GND (black)" (shape input) (at 147.32 52.07 0) (fields_autoplaced)
     (effects (font (size 1.27 1.27)) (justify left))
-    (property "Intersheetrefs" "${INTERSHEET_REFS}" (at 158.7719 52.07 0)
+    (property "Intersheetrefs" "${INTERSHEET_REFS}" (at 166.5128 52.07 0)
       (effects (font (size 1.27 1.27)) (justify left) hide)
     )
   )
-  (global_label "B - D-" (shape input) (at 147.32 91.44 0) (fields_autoplaced)
+  (global_label "B - D-b(white)" (shape input) (at 147.32 91.44 0) (fields_autoplaced)
     (effects (font (size 1.27 1.27)) (justify left))
-    (property "Intersheetrefs" "${INTERSHEET_REFS}" (at 157.9252 91.44 0)
+    (property "Intersheetrefs" "${INTERSHEET_REFS}" (at 165.6662 91.44 0)
       (effects (font (size 1.27 1.27)) (justify left) hide)
     )
   )
-  (global_label "A - 5V" (shape input) (at 147.32 55.88 0) (fields_autoplaced)
+  (global_label "A - 5V (red)" (shape input) (at 147.32 55.88 0) (fields_autoplaced)
     (effects (font (size 1.27 1.27)) (justify left))
-    (property "Intersheetrefs" "${INTERSHEET_REFS}" (at 157.1995 55.88 0)
+    (property "Intersheetrefs" "${INTERSHEET_REFS}" (at 162.8843 55.88 0)
       (effects (font (size 1.27 1.27)) (justify left) hide)
     )
   )
-  (global_label "B - Shield" (shape input) (at 147.32 80.01 0) (fields_autoplaced)
+  (global_label "B - Shield (blue)" (shape input) (at 147.32 80.01 0) (fields_autoplaced)
     (effects (font (size 1.27 1.27)) (justify left))
-    (property "Intersheetrefs" "${INTERSHEET_REFS}" (at 160.9489 80.01 0)
+    (property "Intersheetrefs" "${INTERSHEET_REFS}" (at 167.6617 80.01 0)
       (effects (font (size 1.27 1.27)) (justify left) hide)
     )
   )
-  (global_label "A - Shield" (shape input) (at 147.32 48.26 0) (fields_autoplaced)
+  (global_label "A - Shield (blue)" (shape input) (at 147.32 48.26 0) (fields_autoplaced)
     (effects (font (size 1.27 1.27)) (justify left))
-    (property "Intersheetrefs" "${INTERSHEET_REFS}" (at 160.7675 48.26 0)
+    (property "Intersheetrefs" "${INTERSHEET_REFS}" (at 167.4803 48.26 0)
       (effects (font (size 1.27 1.27)) (justify left) hide)
     )
   )
-  (global_label "B - ID" (shape input) (at 147.32 99.06 0) (fields_autoplaced)
+  (global_label "B - ID (yellow)" (shape input) (at 147.32 99.06 0) (fields_autoplaced)
     (effects (font (size 1.27 1.27)) (justify left))
-    (property "Intersheetrefs" "${INTERSHEET_REFS}" (at 156.9576 99.06 0)
+    (property "Intersheetrefs" "${INTERSHEET_REFS}" (at 165.4847 99.06 0)
       (effects (font (size 1.27 1.27)) (justify left) hide)
     )
   )
-  (global_label "A - D+" (shape input) (at 147.32 63.5 0) (fields_autoplaced)
+  (global_label "A - D+ (green)" (shape input) (at 147.32 63.5 0) (fields_autoplaced)
     (effects (font (size 1.27 1.27)) (justify left))
-    (property "Intersheetrefs" "${INTERSHEET_REFS}" (at 157.7438 63.5 0)
+    (property "Intersheetrefs" "${INTERSHEET_REFS}" (at 165.6662 63.5 0)
       (effects (font (size 1.27 1.27)) (justify left) hide)
     )

Commit message: WIP
Parts:
- added H1, H2, H3, H4: MountingHole, MountingHole:MountingHole_3.2mm_M3, symbol Mechanical:MountingHole
- added J1, J2: Conn_01x06, Connector_JST:JST_XH_S6B-XH-A_1x06_P2.50mm_Horizontal, symbol Connector_Generic:Conn_01x06
- BZ1: footprint (none) -> Buzzer_Beeper:Buzzer_12x9.5RM7.6
Connections:
- net A - 5V (red): now also U1.J4_6 (G21), J1.4 (Pin_4); no longer U1.J4_2 (G23)
- net A - D+ (green): now also U1.J5_12 (G33), J1.2 (Pin_2); no longer U1.J5_13 (G32)
- net A - D- (white): now also U1.J4_3 (G22), J1.3 (Pin_3); no longer U1.J5_8 (G14)
- net A - GND (black): now also U1.J4_8 (G19), J1.5 (Pin_5); no longer U1.J4_9 (G18)
- net A - ID (yellow): now also U1.J4_2 (G23), J1.1 (Pin_1); no longer U1.J4_13 (G4)
- net A - Shield (blue): now also U1.J4_9 (G18), J1.6 (Pin_6); no longer U1.J4_12 (G16)
- net B - 5V (red): now also U1.J4_11 (G17), J2.4 (Pin_4); no longer U1.J5_5 (G13)
- net B - D+ (green): now also U1.J5_11 (G25), J2.2 (Pin_2); no longer U1.J5_12 (G33)
- net B - D-b(white): now also U1.J5_5 (G13), J2.3 (Pin_3); no longer U1.J5_9 (G27)
- net B - GND (black): now also U1.J4_12 (G16), J2.5 (Pin_5); no longer U1.J4_8 (G19)
- net B - ID (yellow): now also J2.1 (Pin_1)
- net B - Shield (blue): now also U1.J4_13 (G4), J2.6 (Pin_6); no longer U1.J4_11 (G17)
- net GND: now reaches BZ1.1 (-), U1.J4_1 (GND_J4_1), U1.J4_7 (GND_J4_7), U1.J5_6 (GND_J5_6), U2.1 (GND)
- net at BZ1.2 (+): now also U1.J5_13 (G32); no longer U1.J5_11 (G25)
- net at U2.3 (SCL): now also U1.J5_8 (G14); no longer U1.J4_3 (G22)
- net at U2.4 (SDA): now also U1.J5_9 (G27); no longer U1.J4_6 (G21)
- net +5V: now reaches U1.J5_1 (5V), U2.2 (VCC_IN)
Other:
- company: (none) -> Sternenlabor e.V.
- title: (none) -> USB Breakout Test Jig
- moved on the sheet: BZ1, U1, U2
