File: Hardware/USB_Breakout_Test_Jig/USB_Breakout_Test_Jig.kicad_sch (KiCad schematic)
At the start: 9 parts, among them J1 Conn_01x06, J2 Conn_01x06, U1 ESP32_NODEMCU, U2 DM-OLED096-636

Commit message: v1.0
Connections:
- net B - D-b(white) renamed B - D- (white)
Changed lines of the file:
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@@
 	(wire
 		(pts
-			(xy 219.71 67.31) (xy 219.71 85.09)
-		)
-		(stroke
-			(width 0)
-			(type default)
-		)
-	)
-	(wire
-		(pts
-			(xy 218.44 97.79) (xy 209.55 97.79)
+			(xy 220.98 67.31) (xy 220.98 85.09)
+		)
+		(stroke
+			(width 0)
+			(type default)
+		)
+	)
+	(wire
+		(pts
+			(xy 219.71 97.79) (xy 209.55 97.79)
 		)
 		(stroke
@@
 	(wire
 		(pts
-			(xy 228.6 52.07) (xy 232.41 52.07)
-		)
-		(stroke
-			(width 0)
-			(type default)
-		)
-	)
-	(wire
-		(pts
-			(xy 219.71 85.09) (xy 209.55 85.09)
+			(xy 214.63 52.07) (xy 232.41 52.07)
+		)
+		(stroke
+			(width 0)
+			(type default)
+		)
+	)
+	(wire
+		(pts
+			(xy 220.98 85.09) (xy 209.55 85.09)
 		)
 		(stroke
@@
 	(wire
 		(pts
-			(xy 224.79 48.26) (xy 232.41 48.26)
-		)
-		(stroke
-			(width 0)
-			(type default)
-		)
-	)
-	(wire
-		(pts
-			(xy 209.55 77.47) (xy 228.6 77.47)
+			(xy 213.36 48.26) (xy 232.41 48.26)
+		)
+		(stroke
+			(width 0)
+			(type default)
+		)
+	)
+	(wire
+		(pts
+			(xy 209.55 77.47) (xy 214.63 77.47)
 		)
 		(stroke
@@
 	(wire
 		(pts
-			(xy 232.41 99.06) (xy 228.6 99.06)
-		)
-		(stroke
-			(width 0)
-			(type default)
-		)
-	)
-	(wire
-		(pts
-			(xy 229.87 83.82) (xy 232.41 83.82)
-		)
-		(stroke
-			(width 0)
-			(type default)
-		)
-	)
-	(wire
-		(pts
-			(xy 223.52 118.11) (xy 223.52 80.01)
-		)
-		(stroke
-			(width 0)
-			(type default)
-		)
-	)
-	(wire
-		(pts
-			(xy 153.67 121.92) (xy 217.17 121.92)
+			(xy 232.41 99.06) (xy 226.06 99.06)
+		)
+		(stroke
+			(width 0)
+			(type default)
+		)
+	)
+	(wire
+		(pts
+			(xy 226.06 83.82) (xy 232.41 83.82)
+		)
+		(stroke
+			(width 0)
+			(type default)
+		)
+	)
+	(wire
+		(pts
+			(xy 222.25 118.11) (xy 222.25 80.01)
+		)
+		(stroke
+			(width 0)
+			(type default)
+		)
+	)
+	(wire
+		(pts
+			(xy 153.67 121.92) (xy 218.44 121.92)
 		)
 		(stroke
@@
 	(wire
 		(pts
-			(xy 163.83 118.11) (xy 223.52 118.11)
+			(xy 163.83 118.11) (xy 222.25 118.11)
 		)
 		(stroke
@@
 	(wire
 		(pts
-			(xy 218.44 63.5) (xy 218.44 97.79)
+			(xy 219.71 63.5) (xy 219.71 97.79)
 		)
 		(stroke
@@
 	(wire
 		(pts
-			(xy 215.9 123.19) (xy 165.1 123.19)
+			(xy 224.79 123.19) (xy 165.1 123.19)
 		)
 		(stroke
@@
 	(wire
 		(pts
-			(xy 226.06 72.39) (xy 226.06 87.63)
+			(xy 224.79 72.39) (xy 224.79 87.63)
 		)
 		(stroke
@@
 	(wire
 		(pts
-			(xy 215.9 91.44) (xy 215.9 123.19)
-		)
-		(stroke
-			(width 0)
-			(type default)
-		)
-	)
-	(wire
-		(pts
-			(xy 228.6 99.06) (xy 228.6 119.38)
-		)
-		(stroke
-			(width 0)
-			(type default)
-		)
-	)
-	(wire
-		(pts
-			(xy 209.55 69.85) (xy 229.87 69.85)
-		)
-		(stroke
-			(width 0)
-			(type default)
-		)
-	)
-	(wire
-		(pts
-			(xy 224.79 74.93) (xy 224.79 48.26)
+			(xy 224.79 91.44) (xy 224.79 123.19)
+		)
+		(stroke
+			(width 0)
+			(type default)
+		)
+	)
+	(wire
+		(pts
+			(xy 226.06 99.06) (xy 226.06 119.38)
+		)
+		(stroke
+			(width 0)
+			(type default)
+		)
+	)
+	(wire
+		(pts
+			(xy 209.55 69.85) (xy 226.06 69.85)
+		)
+		(stroke
+			(width 0)
+			(type default)
+		)
+	)
+	(wire
+		(pts
+			(xy 213.36 74.93) (xy 213.36 48.26)
 		)
 		(stroke
@@
 	(wire
 		(pts
-			(xy 214.63 55.88) (xy 214.63 80.01)
-		)
-		(stroke
-			(width 0)
-			(type default)
-		)
-	)
-	(wire
-		(pts
-			(xy 209.55 87.63) (xy 222.25 87.63)
+			(xy 215.9 55.88) (xy 215.9 80.01)
+		)
+		(stroke
+			(width 0)
+			(type default)
+		)
+	)
+	(wire
+		(pts
+			(xy 209.55 87.63) (xy 220.98 87.63)
 		)
 		(stroke
@@
 	(wire
 		(pts
-			(xy 209.55 80.01) (xy 214.63 80.01)
-		)
-		(stroke
-			(width 0)
-			(type default)
-		)
-	)
-	(wire
-		(pts
-			(xy 226.06 87.63) (xy 232.41 87.63)
+			(xy 209.55 80.01) (xy 215.9 80.01)
+		)
+		(stroke
+			(width 0)
+			(type default)
+		)
+	)
+	(wire
+		(pts
+			(xy 224.79 87.63) (xy 232.41 87.63)
 		)
 		(stroke
@@
 	(wire
 		(pts
-			(xy 223.52 80.01) (xy 232.41 80.01)
-		)
-		(stroke
-			(width 0)
-			(type default)
-		)
-	)
-	(wire
-		(pts
-			(xy 215.9 82.55) (xy 215.9 59.69)
-		)
-		(stroke
-			(width 0)
-			(type default)
-		)
-	)
-	(wire
-		(pts
-			(xy 228.6 119.38) (xy 162.56 119.38)
+			(xy 222.25 80.01) (xy 232.41 80.01)
+		)
+		(stroke
+			(width 0)
+			(type default)
+		)
+	)
+	(wire
+		(pts
+			(xy 217.17 82.55) (xy 217.17 59.69)
+		)
+		(stroke
+			(width 0)
+			(type default)
+		)
+	)
+	(wire
+		(pts
+			(xy 226.06 119.38) (xy 162.56 119.38)
 		)
 		(stroke
@@
 	(wire
 		(pts
-			(xy 209.55 64.77) (xy 217.17 64.77)
+			(xy 209.55 64.77) (xy 218.44 64.77)
 		)
 		(stroke
@@
 	(wire
 		(pts
-			(xy 209.55 72.39) (xy 226.06 72.39)
-		)
-		(stroke
-			(width 0)
-			(type default)
-		)
-	)
-	(wire
-		(pts
-			(xy 222.25 87.63) (xy 222.25 95.25)
+			(xy 209.55 72.39) (xy 224.79 72.39)
+		)
+		(stroke
+			(width 0)
+			(type default)
+		)
+	)
+	(wire
+		(pts
+			(xy 220.98 87.63) (xy 220.98 95.25)
 		)
 		(stroke
@@
 	(wire
 		(pts
-			(xy 218.44 63.5) (xy 232.41 63.5)
+			(xy 219.71 63.5) (xy 232.41 63.5)
 		)
 		(stroke
@@
 	(wire
 		(pts
-			(xy 222.25 95.25) (xy 232.41 95.25)
-		)
-		(stroke
-			(width 0)
-			(type default)
-		)
-	)
-	(wire
-		(pts
-			(xy 229.87 69.85) (xy 229.87 83.82)
+			(xy 220.98 95.25) (xy 232.41 95.25)
+		)
+		(stroke
+			(width 0)
+			(type default)
+		)
+	)
+	(wire
+		(pts
+			(xy 226.06 69.85) (xy 226.06 83.82)
 		)
 		(stroke
@@
 	(wire
 		(pts
-			(xy 215.9 91.44) (xy 232.41 91.44)
-		)
-		(stroke
-			(width 0)
-			(type default)
-		)
-	)
-	(wire
-		(pts
-			(xy 217.17 64.77) (xy 217.17 121.92)
+			(xy 224.79 91.44) (xy 232.41 91.44)
+		)
+		(stroke
+			(width 0)
+			(type default)
+		)
+	)
+	(wire
+		(pts
+			(xy 218.44 64.77) (xy 218.44 121.92)
 		)
 		(stroke
@@
 	(wire
 		(pts
-			(xy 214.63 55.88) (xy 232.41 55.88)
+			(xy 215.9 55.88) (xy 232.41 55.88)
 		)
 		(stroke
@@
 	(wire
 		(pts
-			(xy 228.6 52.07) (xy 228.6 77.47)
+			(xy 214.63 52.07) (xy 214.63 77.47)
 		)
 		(stroke
@@
 	(wire
 		(pts
-			(xy 209.55 74.93) (xy 224.79 74.93)
+			(xy 209.55 74.93) (xy 213.36 74.93)
 		)
 		(stroke
@@
 	(wire
 		(pts
-			(xy 215.9 59.69) (xy 232.41 59.69)
+			(xy 217.17 59.69) (xy 232.41 59.69)
 		)
 		(stroke
@@
 	(wire
 		(pts
-			(xy 215.9 82.55) (xy 209.55 82.55)
+			(xy 217.17 82.55) (xy 209.55 82.55)
 		)
 		(stroke
@@
 	(wire
 		(pts
-			(xy 219.71 67.31) (xy 232.41 67.31)
+			(xy 220.98 67.31) (xy 232.41 67.31)
 		)
 		(stroke
@@
 		)
 	)
-	(global_label "B - D-b(white)"
+	(global_label "B - D- (white)"
 		(shape input)
 		(at 55.88 87.63 0)
@@
 		)
 		(property "Intersheetrefs" "${INTERSHEET_REFS}"
-			(at 74.2262 87.63 0)
+			(at 74.0448 87.63 0)
 			(effects
 				(font
@@
 		)
 	)
-	(global_label "B - D-b(white)"
+	(global_label "B - D- (white)"
 		(shape input)
 		(at 232.41 91.44 0)
@@
 		)
 		(property "Intersheetrefs" "${INTERSHEET_REFS}"
-			(at 250.7562 91.44 0)
-			(effects
-				(font
+			(at 250.5748 91.44 0)
+			(effects
+				(font
